File: MateLightScrewCap.kicad_sch (KiCad schematic)
At the start: 5 parts

Commit message: Small improvements
Parts:
- LD1: value (none) -> APA102; footprint (none) -> MateLightScrewCap:APA102C-5050
- X1: value (none) -> IN; footprint (none) -> h8-Connectors:JST_S2B-ZR-SM4A-TF(LF)(SN)
- X2: value (none) -> OUT; footprint (none) -> h8-Connectors:JST_S2B-ZR-SM4A-TF(LF)(SN)
- X3: value (none) -> Power; footprint (none) -> h8-Connectors:JST_S2B-PH-SM4-TB(LF)(SN)
- X4: value (none) -> Power; footprint (none) -> h8-Connectors:JST_S2B-ZR-SM4A-TF(LF)(SN)
Changed lines of the file:
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@@
       (effects (font (size 1.27 1.27)) hide)
     )
-    (property "Value" "" (id 1) (at 130.81 74.93 90)
+    (property "Value" "+5V" (id 1) (at 130.81 74.93 90)
       (effects (font (size 1.4986 1.4986)) (justify right top))
     )
@@
       (effects (font (size 1.27 1.27)) hide)
     )
-    (property "Value" "" (id 1) (at 124.46 87.63 0)
+    (property "Value" "GND" (id 1) (at 124.46 87.63 0)
       (effects (font (size 1.4986 1.4986)) (justify bottom))
     )
@@
       (effects (font (size 1.27 1.27)) hide)
     )
-    (property "Value" "" (id 1) (at 161.29 115.57 0)
+    (property "Value" "GND" (id 1) (at 161.29 115.57 0)
       (effects (font (size 1.4986 1.4986)) (justify left bottom) hide)
     )
@@
       (effects (font (size 1.4986 1.4986)) (justify left bottom))
     )
-    (property "Value" "" (id 1) (at 143.51 115.57 0)
+    (property "Value" "APA102" (id 1) (at 143.51 115.57 0)
       (effects (font (size 1.4986 1.4986)) (justify left bottom))
     )
-    (property "Footprint" "" (id 2) (at 151.13 102.87 0)
+    (property "Footprint" "MateLightScrewCap:APA102C-5050" (id 2) (at 151.13 102.87 0)
       (effects (font (size 1.27 1.27)) hide)
     )
@@
     (in_bom yes) (on_board yes)
     (property "Reference" "X3" (id 0) (at 110.0328 74.295 0))
-    (property "Value" "" (id 1) (at 110.0328 76.6064 0))
-    (property "Footprint" "" (id 2) (at 107.95 82.55 0)
+    (property "Value" "Power" (id 1) (at 110.0328 76.6064 0))
+    (property "Footprint" "h8-Connectors:JST_S2B-PH-SM4-TB(LF)(SN)" (id 2) (at 107.95 82.55 0)
       (effects (font (size 1.27 1.27)) hide)
     )
@@
     (in_bom yes) (on_board yes)
     (property "Reference" "X1" (id 0) (at 97.3328 97.3582 0))
-    (property "Value" "" (id 1) (at 97.3328 99.6696 0))
-    (property "Footprint" "" (id 2) (at 95.25 102.87 0)
+    (property "Value" "IN" (id 1) (at 97.3328 99.6696 0))
+    (property "Footprint" "h8-Connectors:JST_S2B-ZR-SM4A-TF(LF)(SN)" (id 2) (at 95.25 102.87 0)
       (effects (font (size 1.27 1.27)) hide)
     )
@@
       (effects (font (size 1.27 1.27)) (justify left))
     )
-    (property "Value" "" (id 1) (at 209.042 105.3846 0)
+    (property "Value" "OUT" (id 1) (at 209.042 105.3846 0)
       (effects (font (size 1.27 1.27)) (justify left))
     )
-    (property "Footprint" "" (id 2) (at 207.01 102.87 0)
+    (property "Footprint" "h8-Connectors:JST_S2B-ZR-SM4A-TF(LF)(SN)" (id 2) (at 207.01 102.87 0)
       (effects (font (size 1.27 1.27)) hide)
     )
@@
     (in_bom yes) (on_board yes)
     (property "Reference" "X4" (id 0) (at 97.3328 74.295 0))
-    (property "Value" "" (id 1) (at 97.3328 76.6064 0))
-    (property "Footprint" "" (id 2) (at 95.25 82.55 0)
+    (property "Value" "Power" (id 1) (at 97.3328 76.6064 0))
+    (property "Footprint" "h8-Connectors:JST_S2B-ZR-SM4A-TF(LF)(SN)" (id 2) (at 95.25 82.55 0)
       (effects (font (size 1.27 1.27)) hide)
     )
@@
       (effects (font (size 1.27 1.27)) hide)
     )
-    (property "Value" "" (id 1) (at 166.37 95.25 90)
+    (property "Value" "+5V" (id 1) (at 166.37 95.25 90)
       (effects (font (size 1.4986 1.4986)) (justify left bottom))
     )
